File: Hardware/SparkFun Qwiic Adapter.sch (EAGLE design)
At the start: 6 parts, among them J1 JST, J3 JST, J4 PTH

Commit message: post design review commit
Parts:
- added FD1, FD2, FD3, FD4: FIDUCIALUFIDUCIAL, SparkFun-Aesthetics:FIDUCIALUFIDUCIAL
- added LOGO1: REVISION, SparkFun-Aesthetics:REVISION
- J1, J3: value JST -> (none); device SparkX:I2C_STANDARDJS-1MM -> SparkFun-Connectors:QWIIC_CONNECTORJS-1MM
- J4: device SparkX:I2C_STANDARD_NO_SILK -> SparkFun-Connectors:I2C_STANDARD
- U$1: value SPARKX-LOGO2 -> SFE_LOGO_FLAME.1_INCH; device SparkX:SPARKX-LOGO2 -> SparkFun-Aesthetics:SFE_LOGO_FLAME.1_INCH
Connections:
- net 3.3V: now also J1.2, J3.2, J4.2; no longer J1.VCC, J3.VCC, J4.VCC
- net GND: now also J1.1, J3.1, J4.1; no longer J1.GND, J3.GND, J4.GND
- net SCL: now also J1.4, J3.4, J4.4; no longer J1.SCL, J3.SCL, J4.SCL
- net SDA: now also J1.3, J3.3, J4.3; no longer J1.SDA, J3.SDA, J4.SDA
Other:
- note added: "Andy England"
- note added: "v10"
- note removed: "X10"
