File: Hardware/SparkFun Qwiic Adapter.brd (EAGLE design)
At the start: 22.9 x 7.6 mm, 6 parts, among them J1 JST, J3 JST, J4 PTH

Commit message: post design review commit
Parts:
- added FD1, FD2, FD3, FD4: FIDUCIALUFIDUCIAL, SparkFun-Aesthetics:FIDUCIAL-MICRO
- added LOGO1: REVISION, SparkFun-Aesthetics:REVISION
- J1, J3: value JST -> (none); device SparkX:1X04_1MM_RA -> SparkFun-Connectors:1X04_1MM_RA
- J4: device SparkX:1X04_NO_SILK -> SparkFun-Connectors:1X04
- U$1: value SPARKX-LOGO2 -> SFE_LOGO_FLAME.1_INCH; device SparkX:SPARKX-TINY -> SparkFun-Aesthetics:SFE_LOGO_FLAME_.1
- moved FRAME1 13.0 mm to (-16.5, -8.89)
- moved U$1 1.80 mm to (4.45, 2.54)
Other:
- board text added: "Andy England"
- board text added: "v10"
Changed lines of the file:
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@@
 <layer number="45" name="Holes" color="7" fill="1" visible="yes" active="yes"/>
 <layer number="46" name="Milling" color="3" fill="1" visible="no" active="yes"/>
-<layer number="47" name="Measures" color="7" fill="1" visible="no" active="yes"/>
+<layer number="47" name="Measures" color="7" fill="1" visible="yes" active="yes"/>
 <layer number="48" name="Document" color="7" fill="1" visible="no" active="yes"/>
 <layer number="49" name="Reference" color="7" fill="1" visible="no" active="yes"/>
@@
 <layer number="230" name="230bmp" color="7" fill="1" visible="no" active="yes"/>
 <layer number="231" name="231bmp" color="7" fill="1" visible="no" active="yes"/>
+<layer number="232" name="Eagle3D_PG2" color="7" fill="1" visible="yes" active="yes"/>
+<layer number="233" name="Eagle3D_PG3" color="7" fill="1" visible="yes" active="yes"/>
 <layer number="248" name="Housing" color="7" fill="1" visible="no" active="yes"/>
 <layer number="249" name="Edge" color="7" fill="1" visible="no" active="yes"/>
@@
 <text x="12.7" y="3.81" size="1.016" layer="22" font="vector" ratio="15" rot="MR270" align="center-left">3.3V</text>
 <text x="15.24" y="3.81" size="1.016" layer="22" font="vector" ratio="15" rot="MR270" align="center-left">GND</text>
-<text x="16.51" y="-21.59" size="1.778" layer="51">Nathan Seidle</text>
+<text x="13.97" y="-8.89" size="1.778" layer="51">Nathan Seidle</text>
+<text x="22.479" y="0.381" size="1.27" layer="16" font="vector" ratio="20" rot="MR0">v10</text>
+<text x="13.97" y="-11.43" size="1.778" layer="51" font="vector">Andy England</text>
+<dimension x1="0" y1="7.62" x2="22.86" y2="7.62" x3="11.43" y3="10.16" textsize="1.778" layer="47" unit="inch"/>
+<dimension x1="0" y1="0" x2="0" y2="7.62" x3="-2.54" y3="3.81" textsize="1.778" layer="47" unit="inch"/>
 </plain>
 <attributes>
@@
 </class>
 </classes>
-<designrules name="SparkFun-2-layer-STANDARD">
+<designrules name="SparkFun-2-layer-TIGHT">
 <description language="en">&lt;b&gt;SparkFun 2 Layer Design Rule Checks - STANDARD/TIGHT/FAB-LIMIT&lt;/b&gt;
 &lt;p&gt;
@@
 <param name="mtCopper" value="0.035mm 0.035mm 0.035mm 0.035mm 0.035mm 0.035mm 0.035mm 0.035mm 0.035mm 0.035mm 0.035mm 0.035mm 0.035mm 0.035mm 0.035mm 0.035mm"/>
 <param name="mtIsolate" value="1.5mm 0.15mm 0.2mm 0.15mm 0.2mm 0.15mm 0.2mm 0.15mm 0.2mm 0.15mm 0.2mm 0.15mm 0.2mm 0.15mm 0.2mm"/>
-<param name="mdWireWire" value="10mil"/>
-<param name="mdWirePad" value="8mil"/>
-<param name="mdWireVia" value="10mil"/>
-<param name="mdPadPad" value="8mil"/>
-<param name="mdPadVia" value="10mil"/>
-<param name="mdViaVia" value="10mil"/>
-<param name="mdSmdPad" value="8mil"/>
-<param name="mdSmdVia" value="8mil"/>
-<param name="mdSmdSmd" value="8mil"/>
+<param name="mdWireWire" value="7mil"/>
+<param name="mdWirePad" value="7mil"/>
+<param name="mdWireVia" value="7mil"/>
+<param name="mdPadPad" value="7mil"/>
+<param name="mdPadVia" value="7mil"/>
+<param name="mdViaVia" value="7mil"/>
+<param name="mdSmdPad" value="7mil"/>
+<param name="mdSmdVia" value="7mil"/>
+<param name="mdSmdSmd" value="7mil"/>
 <param name="mdViaViaSameLayer" value="8mil"/>
 <param name="mnLayersViaInSmd" value="2"/>
-<param name="mdCopperDimension" value="8mil"/>
-<param name="mdDrill" value="8mil"/>
+<param name="mdCopperDimension" value="7mil"/>
+<param name="mdDrill" value="7mil"/>
 <param name="mdSmdStop" value="0mil"/>
-<param name="msWidth" value="10mil"/>
-<param name="msDrill" value="20mil"/>
+<param name="msWidth" value="7mil"/>
+<param name="msDrill" value="15mil"/>
 <param name="msMicroVia" value="9.99mm"/>
 <param name="msBlindViaRatio" value="0.5"/>
@@
 <param name="rvMicroViaOuter" value="0.25"/>
 <param name="rvMicroViaInner" value="0.25"/>
-<param name="rlMinPadTop" value="10mil"/>
+<param name="rlMinPadTop" value="7mil"/>
 <param name="rlMaxPadTop" value="20mil"/>
-<param name="rlMinPadInner" value="10mil"/>
+<param name="rlMinPadInner" value="7mil"/>
 <param name="rlMaxPadInner" value="20mil"/>
-<param name="rlMinPadBottom" value="10mil"/>
+<param name="rlMinPadBottom" value="7mil"/>
 <param name="rlMaxPadBottom" value="20mil"/>
-<param name="rlMinViaOuter" value="10mil"/>
+<param name="rlMinViaOuter" value="7mil"/>
 <param name="rlMaxViaOuter" value="20mil"/>
-<param name="rlMinViaInner" value="10mil"/>
+<param name="rlMinViaInner" value="7mil"/>
 <param name="rlMaxViaInner" value="20mil"/>
 <param name="rlMinMicroViaOuter" value="4mil"/>
@@
 </autorouter>
 <elements>
-<element name="FRAME1" library="SparkFun-Aesthetics" package="CREATIVE_COMMONS" value="FRAME-LETTER" x="-13.97" y="-21.59"/>
+<element name="FRAME1" library="SparkFun-Aesthetics" package="CREATIVE_COMMONS" value="FRAME-LETTER" x="-16.51" y="-8.89"/>
 <element name="LOGO4" library="SparkFun-Aesthetics" package="OSHW-LOGO-S" value="OSHW-LOGOS" x="20.32" y="3.81" rot="MR0"/>
-<element name="U$1" library="SparkX" package="SPARKX-TINY" value="SPARKX-LOGO2" x="3.175" y="3.81" rot="MR0"/>
-<element name="J3" library="SparkX" package="1X04_1MM_RA" value="JST" x="17.78" y="3.81" rot="R90"/>
-<element name="J4" library="SparkX" package="1X04_NO_SILK" value="PTH" x="15.24" y="5.08" rot="R180"/>
-<element name="J1" library="SparkX" package="1X04_1MM_RA" value="JST" x="5.08" y="3.81" rot="R270"/>
+<element name="U$1" library="SparkFun-Aesthetics" package="SFE_LOGO_FLAME_.1" value="SFE_LOGO_FLAME.1_INCH" x="4.445" y="2.54" rot="MR0"/>
+<element name="J3" library="SparkFun-Connectors" package="1X04_1MM_RA" value="" x="17.78" y="3.81" rot="R90">
+<attribute name="PROD_ID" value="CONN-13694" x="17.78" y="3.81" size="1.778" layer="27" rot="R90" display="off"/>
+<attribute name="VALUE" value="" x="17.78" y="3.81" size="1.778" layer="27" rot="R90" display="off"/>
+</element>
+<element name="J4" library="SparkFun-Connectors" package="1X04" value="PTH" x="15.24" y="5.08" rot="R180"/>
+<element name="J1" library="SparkFun-Connectors" package="1X04_1MM_RA" value="" x="5.08" y="3.81" rot="R270">
+<attribute name="PROD_ID" value="CONN-13694" x="5.08" y="3.81" size="1.778" layer="27" rot="R270" display="off"/>
+<attribute name="VALUE" value="" x="5.08" y="3.81" size="1.778" layer="27" rot="R270" display="off"/>
+</element>
+<element name="FD1" library="SparkFun-Aesthetics" package="FIDUCIAL-MICRO" value="FIDUCIALUFIDUCIAL" x="8.89" y="2.54"/>
+<element name="FD2" library="SparkFun-Aesthetics" package="FIDUCIAL-MICRO" value="FIDUCIALUFIDUCIAL" x="8.89" y="2.54" rot="MR0"/>
+<element name="FD3" library="SparkFun-Aesthetics" package="FIDUCIAL-MICRO" value="FIDUCIALUFIDUCIAL" x="13.97" y="3.81"/>
+<element name="FD4" library="SparkFun-Aesthetics" package="FIDUCIAL-MICRO" value="FIDUCIALUFIDUCIAL" x="13.97" y="3.81" rot="MR0"/>
+<element name="LOGO1" library="SparkFun-Aesthetics" package="REVISION" value="REVISION" x="-5.08" y="-11.43"/>
 </elements>
 <signals>
@@
 <wire x1="15.597" y1="2.31" x2="15.24" y2="2.667" width="0.3048" layer="1"/>
 <wire x1="15.24" y1="2.667" x2="15.24" y2="5.08" width="0.3048" layer="1"/>
-<via x="6.35" y="6.731" extent="1-16" drill="0.381"/>
 <wire x1="6.35" y1="6.731" x2="14.732" y2="6.731" width="0.3048" layer="16"/>
 <wire x1="14.732" y1="6.731" x2="15.24" y2="6.223" width="0.3048" layer="16"/>
@@
 <wire x1="5.08" y1="6.223" x2="5.588" y2="6.731" width="0.3048" layer="1"/>
 <wire x1="5.588" y1="6.731" x2="6.35" y2="6.731" width="0.3048" layer="1"/>
+<via x="6.35" y="6.731" extent="1-16" drill="0.381"/>
 </signal>
 <signal name="SCL">

Commit message: Checklist changes
Parts:
- moved U$1 1.67 mm to (2.79, 2.79), turned to 90 degrees
- moved FD3 0.64 mm to (14.0, 3.17)
- moved FD4 0.64 mm to (14.0, 3.17)
Other:
- board text added: "Qwiic Adapter"
Changed lines of the file:
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@@
 <board>
 <plain>
-<wire x1="0" y1="0" x2="0" y2="7.62" width="0.3048" layer="20"/>
-<wire x1="0" y1="7.62" x2="22.86" y2="7.62" width="0.3048" layer="20"/>
-<wire x1="22.86" y1="7.62" x2="22.86" y2="0" width="0.3048" layer="20"/>
-<wire x1="22.86" y1="0" x2="0" y2="0" width="0.3048" layer="20"/>
+<wire x1="0" y1="0" x2="0" y2="7.62" width="0.2032" layer="20"/>
+<wire x1="0" y1="7.62" x2="22.86" y2="7.62" width="0.2032" layer="20"/>
+<wire x1="22.86" y1="7.62" x2="22.86" y2="0" width="0.2032" layer="20"/>
+<wire x1="22.86" y1="0" x2="0" y2="0" width="0.2032" layer="20"/>
 <text x="7.62" y="3.81" size="1.016" layer="21" font="vector" ratio="15" rot="R270" align="center-left">SCL</text>
 <text x="10.16" y="3.81" size="1.016" layer="21" font="vector" ratio="15" rot="R270" align="center-left">SDA</text>
@@
 <dimension x1="0" y1="7.62" x2="22.86" y2="7.62" x3="11.43" y3="10.16" textsize="1.778" layer="47" unit="inch"/>
 <dimension x1="0" y1="0" x2="0" y2="7.62" x3="-2.54" y3="3.81" textsize="1.778" layer="47" unit="inch"/>
+<text x="2.032" y="3.81" size="0.8128" layer="22" font="vector" ratio="15" rot="MR270" align="center">Qwiic
+Adapter</text>
 </plain>
 <attributes>
@@
 <element name="FRAME1" library="SparkFun-Aesthetics" package="CREATIVE_COMMONS" value="FRAME-LETTER" x="-16.51" y="-8.89"/>
 <element name="LOGO4" library="SparkFun-Aesthetics" package="OSHW-LOGO-S" value="OSHW-LOGOS" x="20.32" y="3.81" rot="MR0"/>
-<element name="U$1" library="SparkFun-Aesthetics" package="SFE_LOGO_FLAME_.1" value="SFE_LOGO_FLAME.1_INCH" x="4.445" y="2.54" rot="MR0"/>
+<element name="U$1" library="SparkFun-Aesthetics" package="SFE_LOGO_FLAME_.1" value="SFE_LOGO_FLAME.1_INCH" x="2.794" y="2.794" rot="MR90"/>
 <element name="J3" library="SparkFun-Connectors" package="1X04_1MM_RA" value="" x="17.78" y="3.81" rot="R90">
 <attribute name="PROD_ID" value="CONN-13694" x="17.78" y="3.81" size="1.778" layer="27" rot="R90" display="off"/>
@@
 <element name="FD1" library="SparkFun-Aesthetics" package="FIDUCIAL-MICRO" value="FIDUCIALUFIDUCIAL" x="8.89" y="2.54"/>
 <element name="FD2" library="SparkFun-Aesthetics" package="FIDUCIAL-MICRO" value="FIDUCIALUFIDUCIAL" x="8.89" y="2.54" rot="MR0"/>
-<element name="FD3" library="SparkFun-Aesthetics" package="FIDUCIAL-MICRO" value="FIDUCIALUFIDUCIAL" x="13.97" y="3.81"/>
-<element name="FD4" library="SparkFun-Aesthetics" package="FIDUCIAL-MICRO" value="FIDUCIALUFIDUCIAL" x="13.97" y="3.81" rot="MR0"/>
+<element name="FD3" library="SparkFun-Aesthetics" package="FIDUCIAL-MICRO" value="FIDUCIALUFIDUCIAL" x="13.97" y="3.175"/>
+<element name="FD4" library="SparkFun-Aesthetics" package="FIDUCIAL-MICRO" value="FIDUCIALUFIDUCIAL" x="13.97" y="3.175" rot="MR0"/>
 <element name="LOGO1" library="SparkFun-Aesthetics" package="REVISION" value="REVISION" x="-5.08" y="-11.43"/>
 </elements>
@@
 </board>
 </drawing>
+<compatibility>
+<note version="6.3" minversion="6.2.2" severity="warning">
+Since Version 6.2.2 text objects can contain more than one line,
+which will not be processed correctly with this version.
+</note>
+</compatibility>
 </eagle>
